File: sch/rec_play_switch_module/rec_play_switch_module.kicad_pcb (KiCad board)
At the start: 2 copper layers, 86.6 x 50.3 mm, 25 parts, among them J1 Conn_01x24, J2 Conn_01x12, J3 Conn_02x03_Counter_Clockwise, J4 Conn_01x02, J9 Conn_01x02, K1 G6K-2P-Y, K2 G6K-2P-Y, K3 G6K-2P-Y, K4 G6K-2P-Y, K5 G6K-2P-Y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

Commit message: r2
Parts:
- moved J3 5.68 mm to (146.6, 62.4), turned to 90 degrees
Routing:
- net /MISO: track 38.2 -> 48.4 mm
- net /SCK: track 33.5 -> 39.8 mm
- net +5V: track 109.5 -> 113.2 mm
- net /RESET: track 23.1 -> 26.0 mm
- net /MOSI: track 39.2 -> 38.2 mm
