File: sch/rec_play_switch_module/rec_play_switch_module.kicad_sch (KiCad schematic)
At the start: 25 parts, among them J1 Conn_01x24, J2 Conn_01x12, J3 Conn_02x03_Counter_Clockwise, J4 Conn_01x02, J9 Conn_01x02, K1 G6K-2P-Y, K2 G6K-2P-Y, K3 G6K-2P-Y, K4 G6K-2P-Y, K5 G6K-2P-Y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

Commit message: r2
Connections:
- no-connect marks 9 -> 16
Changed lines of the file:
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@@
+	)
+	(no_connect
+		(at 76.2 172.72)
+	)
+	(no_connect
+		(at 76.2 167.64)
 	)
 	(no_connect
@@
 	(no_connect
 		(at 76.2 152.4)
+	)
+	(no_connect
+		(at 76.2 124.46)
 	)
 	(no_connect
@@
 	)
 	(no_connect
+		(at 76.2 127)
+	)
+	(no_connect
 		(at 76.2 154.94)
 	)
+	(no_connect
+		(at 76.2 175.26)
+	)
+	(no_connect
+		(at 76.2 170.18)
+	)
+	(no_connect
+		(at 76.2 165.1)
+	)
 	(wire
